Commit message: descrption modified

File: bobac2_description/urdf/bobac2_description.urdf (robot description, URDF)
Before this commit: robot bobac2_description, 24 links, 23 joints
Links:
- added link imu_Link, mass 0.01; collision box size=0.02 0.02 0.02; visual box size=0.02 0.02 0.02
Joints:
- added joint imu_joint: type fixed, parent base_link, child imu_Link, origin xyz=0.00 0 0.1 rpy=0 0 0, axis 0 0 0

File: bobac2_description/urdf/gazebo_bobac2_description.urdf (robot description, URDF)
Before this commit: robot bobac2_description, 24 links, 23 joints
Links:
- added link imu_Link, mass 0.01; collision box size=0.02 0.02 0.02; visual box size=0.02 0.02 0.02
Joints:
- added joint imu_joint: type fixed, parent base_link, child imu_Link, origin xyz=0.00 0 0.1 rpy=0 0 0, axis 0 0 0
- joint kinect_optical_joint: origin xyz=0 0 0.29 rpy=-1.5708 0 -1.5708 -> xyz=0 0 -0.01 rpy=-1.5708 0 -1.5708
